File: pcb/smartpoopbucket.kicad_pcb (KiCad board)
At the start: 2 copper layers, 49 x 23 mm, 11 parts, among them U1 XIAO-ESP32-S3-SMD

Commit message: Updated CAD and firmware
Routing:
- net DT: track 38.0 -> 37.4 mm
Other:
- board text added: "while you're here... notice how there's nothing this side of the board? that's SMD for ya!"
Changed lines of the file:
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@@
 			(outputformat 1)
 			(mirror no)
-			(drillshape 1)
+			(drillshape 0)
 			(scaleselection 1)
-			(outputdirectory "")
+			(outputdirectory "gerbers/")
 		)
 	)
@@
 		)
 	)
-	(gr_text "wait! you shouldn't be able to see this!\nhmm... something's gone wrong. either everything in the\nworld has turned upside down or you've...\nvoided your non-existent warranty!"
-		(at 77.6 31.6 0)
+	(gr_text "while you're here... notice how there's \nnothing this side of the board? that's SMD for ya!"
+		(at 75.6 39.9 0)
 		(layer "B.SilkS")
 		(effects
@@
 		)
 	)
+	(gr_text "wait! you shouldn't be able to see this!\nhmm... something's gone wrong. either everything in the\nworld has turned upside down or you've...\nvoided your non-existent warranty!"
+		(at 78.1 31.6 0)
+		(layer "B.SilkS")
+		(effects
+			(font
+				(size 1 1)
+				(thickness 0.1)
+			)
+			(justify left bottom mirror)
+		)
+	)
 	(segment
-		(start 35.4 22.8)
-		(end 35.4 22.9)
+		(start 34.1 24.5)
+		(end 34.1 27.7)
+		(width 0.2)
+		(layer "F.Cu")
+		(net 20)
+	)
+	(segment
+		(start 34.1 27.7)
+		(end 34.34 27.94)
 		(width 0.2)
 		(layer "F.Cu")
@@
 	)
 	(segment
-		(start 34.1 24.2)
-		(end 34.1 27.7)
+		(start 61.6 23.2)
+		(end 35.4 23.2)
 		(width 0.2)
 		(layer "F.Cu")
@@
 	)
 	(segment
-		(start 61.2 22.8)
-		(end 35.4 22.8)
+		(start 35.4 23.2)
+		(end 34.1 24.5)
 		(width 0.2)
 		(layer "F.Cu")
@@
 	)
 	(segment
-		(start 34.1 27.7)
-		(end 34.34 27.94)
+		(start 63.9 25.5)
+		(end 61.6 23.2)
 		(width 0.2)
 		(layer "F.Cu")
@@
 	)
 	(segment
-		(start 63.9 25.5)
-		(end 61.2 22.8)
+		(start 34.9 22.7)
+		(end 33.7 23.9)
 		(width 0.2)
 		(layer "F.Cu")
-		(net 20)
+		(net 21)
 	)
 	(segment
-		(start 35.4 22.9)
-		(end 34.1 24.2)
-		(width 0.2)
-		(layer "F.Cu")
-		(net 20)
-	)
-	(segment
-		(start 65 22.4)
-		(end 35.2 22.4)
+		(start 68.1 25.5)
+		(end 65.3 22.7)
 		(width 0.2)
 		(layer "F.Cu")
@@
 	)
 	(segment
-		(start 35.2 22.4)
-		(end 33.7 23.9)
+		(start 65.3 22.7)
+		(end 34.9 22.7)
 		(width 0.2)
 		(layer "F.Cu")
@@
 	)
 	(segment
-		(start 68.1 25.5)
-		(end 65 22.4)
+		(start 33.88 30.48)
+		(end 36.9 30.48)
 		(width 0.2)
 		(layer "F.Cu")
@@
 		(width 0.2)
 		(layer "F.Cu")
-		(net 21)
-	)
-	(segment
-		(start 33.88 30.48)
-		(end 36.9 30.48)
-		(width 0.2)
-		(layer "F.Cu")
